Commit message: Updated urdf file with Lidar

File: tortoise_ws/src/tortoise_bot/urdf/simple_bot.urdf (robot description, URDF)
Before this commit: robot tbot_v7, 6 links, 5 joints
Links:
- added link lidar_link, mass 0.1; collision cylinder length=0.04 radius=0.03; visual cylinder length=0.04 radius=0.03
Joints:
- added joint lidar_joint: type fixed, parent sensor_mount, child lidar_link, origin xyz=0 0 0.08 rpy=0 0 0

Commit message: 31 July 2025

File: tortoise_ws/src/tortoise_bot/urdf/simple_bot.urdf (robot description, URDF)
Before this commit: robot tbot_v7, 7 links, 6 joints
Links:
- link front_caster: geometry collision sphere radius=0.04; visual sphere radius=0.14

Commit message: Task 02 Completed

File: tortoise_ws/src/tortoise_bot/urdf/simple_bot.urdf (robot description, URDF)
Before this commit: robot tbot_v7, 7 links, 6 joints
Links:
- added link rear_caster, mass 0.25; collision sphere radius=0.08; visual sphere radius=0.08
- link front_caster: mass 0.15 -> 0.25; geometry collision sphere radius=0.08; visual sphere radius=0.08
Joints:
- added joint rear_caster_joint: type fixed, parent base_link, child rear_caster, origin xyz=-0.15 0 -0.06 rpy=0 0 0
- joint battery_joint: origin xyz=-0.05 0 -0.05 rpy=0 0 0 -> xyz=-0 0 -0.05 rpy=0 0 0
- joint front_caster_joint: origin xyz=0.20 0 -0.06 rpy=0 0 0 -> xyz=0.15 0 -0.06 rpy=0 0 0
- joint left_wheel_joint: origin xyz=-0.18 0.175 -0.04 rpy=0 0 0 -> xyz=0 0.175 -0.04 rpy=0 0 0
- joint right_wheel_joint: origin xyz=-0.18 -0.175 -0.04 rpy=0 0 0 -> xyz=0 -0.175 -0.04 rpy=0 0 0
- joint sensor_mount_joint: origin xyz=0.05 0 0.09 rpy=0 0 0 -> xyz=0 0 0.09 rpy=0 0 0
