Commit message: just added ros2_control xacro file to urdf

File: arm_ws/src/arm_description/urdf/arm.urdf copy 2.xacro (robot description, xacro)
@@ -417,11 +417,11 @@
   </link>
   <!-- Connect wrist to gripper base -->
-  <joint name="le_1_to_g_base" type="fixed">
+  <!-- <joint name="le_1_to_g_base" type="fixed">
     <origin rpy="0 0 0" xyz="0 0 0.1"/>
     <parent link="le_1"/>
     <child link="g_base"/>
-  </joint>
+  </joint> -->
   <!-- Gripper base -->
-  <link name="g_base">
+  <!-- <link name="g_base">
     <visual>
       <geometry>
@@ -445,7 +445,7 @@
         izz="0.0025"/>
     </inertial>
-  </link>
+  </link> -->
   <!-- Gripper Right Finger -->
-  <link name="gripper_right_finger">
+  <!-- <link name="gripper_right_finger">
     <visual>
       <geometry>
@@ -469,6 +469,6 @@
         izz="0.00002"/>
     </inertial>
-  </link>
-  <joint name="gripper_right_finger_joint" type="prismatic">
+  </link> -->
+  <!-- <joint name="gripper_right_finger_joint" type="prismatic">
     <axis xyz="0 1 0"/>
     <origin xyz="0.0 -0.07 0.03" rpy="0.0 0.0 0.0"/>
@@ -477,7 +477,7 @@
     <limit effort="100.0" lower="0.0" upper="0.05" velocity="1.0"/>
     <dynamics damping="2.0" friction="1.0"/>
-  </joint>
+  </joint> -->
   <!-- Gripper Left Finger -->
-  <link name="gripper_left_finger">
+  <!-- <link name="gripper_left_finger">
     <visual>
       <geometry>
@@ -501,6 +501,6 @@
         izz="0.00002"/>
     </inertial>
-  </link>
-  <joint name="gripper_left_finger_joint" type="prismatic">
+  </link> -->
+  <!-- <joint name="gripper_left_finger_joint" type="prismatic">
     <axis xyz="0 1 0"/>
     <origin xyz="0.0 0.07 0.03" rpy="0.0 0.0 0.0"/>
@@ -510,12 +510,154 @@
     <dynamics damping="2.0" friction="1.0"/>
     <mimic joint="gripper_right_finger_joint" multiplier="-1.0" offset="0"/>
-  </joint>
+  </joint> -->
   <!-- Tool Center Point (TCP) / End Effector Frame -->
-  <link name="tool0"/>
+  <!-- <link name="tool0"/>
   <joint name="g_base_to_tool0" type="fixed">
     <origin xyz="0 0 0.15" rpy="0 0 0"/>
     <parent link="g_base"/>
     <child link="tool0"/>
-  </joint>
-  <xacro:include filename="six-axis.ros2_control.xacro" />
+  </joint> -->
+  <!-- Ros2_Control -->
+  <!-- <ros2_control name="GazeboSimSystem" type="system">
+    <hardware>
+      <plugin>gz_ros2_control/GazeboSimSystem</plugin>
+    </hardware>
+    <joint name="j1">
+      <command_interface name="position">
+        <param name="min">-6.283185307179586</param>
+        <param name="max">6.283185307179586</param>
+      </command_interface>
+      <command_interface name="velocity">
+        <param name="min">-2.0</param>
+        <param name="max">2.0</param>
+      </command_interface>
+      <state_interface name="position">
+        <param name="initial_value">0.0</param>
+      </state_interface>
+      <state_interface name="velocity"/>
+      <state_interface name="effort"/>
+    </joint>
+    <joint name="j2">
+      <command_interface name="position">
+        <param name="min">-1.5707963267948966</param>
+        <param name="max">1.5707963267948966</param>
+      </command_interface>
+      <command_interface name="velocity">
+        <param name="min">-2.0</param>
+        <param name="max">2.0</param>
+      </command_interface>
+      <state_interface name="position">
+        <param name="initial_value">0.0</param>
+      </state_interface>
+      <state_interface name="velocity"/>
+      <state_interface name="effort"/>
+    </joint>
+    <joint name="j3">
+      <command_interface name="position">
+        <param name="min">-1.5707963267948966</param>
+        <param name="max">1.5707963267948966</param>
+      </command_interface>
+      <command_interface name="velocity">
+        <param name="min">-2.0</param>
+        <param name="max">2.0</param>
+      </command_interface>
+      <state_interface name="position">
+        <param name="initial_value">0.0</param>
+      </state_interface>
+      <state_interface name="velocity"/>
+      <state_interface name="effort"/>
+    </joint>
+    <joint name="j4">
+      <command_interface name="position">
+        <param name="min">-1.5707963267948966</param>
+        <param name="max">1.5707963267948966</param>
+      </command_interface>
+      <command_interface name="velocity">
+        <param name="min">-2.0</param>
+        <param name="max">2.0</param>
+      </command_interface>
+      <state_interface name="position">
+        <param name="initial_value">0.0</param>
+      </state_interface>
+      <state_interface name="velocity"/>
+      <state_interface name="effort"/>
+    </joint>
+    <joint name="j5">
+      <command_interface name="position">
+        <param name="min">-3.141592653589793</param>
+        <param name="max">3.141592653589793</param>
+      </command_interface>
+      <command_interface name="velocity">
+        <param name="min">-2.0</param>
+        <param name="max">2.0</param>
+      </command_interface>
+      <state_interface name="position">
+        <param name="initial_value">0.0</param>
+      </state_interface>
+      <state_interface name="velocity"/>
+      <state_interface name="effort"/>
+    </joint>
+    <joint name="j6">
+      <command_interface name="position">
+        <param name="min">-6.283185307179586</param>
+        <param name="max">6.283185307179586</param>
+      </command_interface>
+      <command_interface name="velocity">
+        <param name="min">-2.0</param>
+        <param name="max">2.0</param>
+      </command_interface>
+      <state_interface name="position">
+        <param name="initial_value">0.0</param>
+      </state_interface>
+      <state_interface name="velocity"/>
+      <state_interface name="effort"/>
+    </joint>
+    <joint name="gripper_right_finger_joint">
+      <command_interface name="position">
+        <param name="min">0.0</param>
+        <param name="max">0.05</param>
+      </command_interface>
+      <state_interface name="position">
+        <param name="initial_value">0.0</param>
+      </state_interface>
+      <state_interface name="velocity"/>
+      <state_interface name="effort"/>
+    </joint>
+    <joint name="gripper_left_finger_joint">
+      <command_interface name="position">
+        <param name="min">-0.05</param>
+        <param name="max">0.0</param>
+      </command_interface>
+      <state_interface name="position">
+        <param name="initial_value">0.0</param>
+      </state_interface>
+      <state_interface name="velocity"/>
+      <state_interface name="effort"/>
+    </joint>
+  </ros2_control> -->
+  <!-- Gazebo Plugins -->
+  <!-- <gazebo>
+    <disableFixedJointLumping>true</disableFixedJointLumping>
+  </gazebo>
+  <gazebo>
+    <plugin filename="gz-sim-joint-state-publisher-system" name="gz::sim::systems::JointStatePublisher">
+      <topic>joint_states</topic>
+      <joint_name>world_joint</joint_name>
+      <joint_name>j1</joint_name>
+      <joint_name>j2</joint_name>
+      <joint_name>j3</joint_name>
+      <joint_name>j4</joint_name>
+      <joint_name>j5</joint_name>
+      <joint_name>j6</joint_name>
+      <joint_name>gripper_left_finger_joint</joint_name>
+      <joint_name>gripper_right_finger_joint</joint_name>
+    </plugin>
+  </gazebo>
+  <gazebo>
+  <plugin filename="libgz_ros2_control-system.so"
+          name="gz_ros2_control::GazeboSimROS2ControlPlugin">
+    <parameters>$(find arm_description)/config/ros2_controllers.yaml</parameters>
+    <controller_manager_node_name>controller_manager</controller_manager_node_name>
+  </plugin>
+</gazebo> -->
 </robot>

File: backups/arm_moveit_config_backup/config/six-axis.ros2_control.xacro (robot description, xacro)
@@ -1,4 +1,6 @@
 <?xml version="1.0"?>
 <robot xmlns:xacro="http://www.ros.org/wiki/xacro">
+    <xacro:macro name="six-axis_ros2_control" params="name initial_positions_file">
+        <xacro:property name="initial_positions" value="${xacro.load_yaml(initial_positions_file)['initial_positions']}"/>
         <ros2_control name="${name}" type="system">
             <hardware>
@@ -48,11 +50,5 @@
                 <state_interface name="velocity"/>
             </joint>
-            <joint name="gripper_right_finger_joint">
-                <command_interface name="position"/>
-                <state_interface name="position">
-                  <param name="initial_value">${initial_positions['gripper_right_finger_joint']}</param>
-                </state_interface>
-                <state_interface name="velocity"/>
-            </joint>
         </ros2_control>
+    </xacro:macro>
 </robot>
