Commit message: upto URDF of ARM is correct

File: arm_ws/src/arm_description/urdf/arm.urdf.xacro (robot description, xacro)
@@ -1,293 +1,663 @@
-<?xml version="1.0"?>
-<robot name="six-axis" xmlns:xacro="http://www.ros.org/wiki/xacro" xmlns:ros2_control="http://www.ros.org/wiki/ros2_control">
-<!-- Define gray color -->
-  <material name="gray">
-   <color rgba="0.75 0.75 0.75 1.0"/>
-  </material>
-<!-- Define silver color -->
-<material name="silver">
-    <!-- <color rgba="0.75 0.75 0.75 1.0"/> -->
-    <color rgba="0.9 0.9 0.98 1.0"/>
-</material>
-<!-- Fixed Link -->
-<link name="base_link"></link>
-<!-- Fixed Joint -->
-<joint name="j0" type="fixed">
-    <origin xyz="0.0 0.0 0.0" rpy="0.0 0.0 0.0"/>
-    <parent link="base_link"/>
-    <child link="l0"/>
-    <axis xyz="0.0 0.0 0.0"/>
-    <limit lower="0.0" upper="0.0" effort="0.0" velocity="0.0"/>
-</joint>
-<link name="l0">
-    <inertial>
-			<origin xyz="0.0 0.0 25e-03" rpy="0 0 0"/>
-			<mass value="2e+00"/>
-			<inertia
-				ixx="9.3895308e-03" ixy="0.0" ixz="1.1882474e-03"
-				iyx="0.0" iyy="1.4207390e-02" iyz="9.2874266e-06"
-				izx="1.1882474e-04"  izy="9.2874266e-06"  izz="1.7661948e-02"/>
-	</inertial>
-    <visual>
-        <geometry>
-            <cylinder radius="0.1" length="0.05"/>
-        </geometry>
-        <origin xyz="0.0 0.0 0.0" rpy="0.0 0.0 0.0"/>
-        <material name="silver"/>
-    </visual>
-</link>
-<joint name="j1" type="revolute">
-    <origin xyz="0.0 0.0 0.0" rpy="0.0 0.0 0.0"/>
-    <parent link="l0"/>
-    <child link="l1"/>
-    <axis xyz="0.0 0.0 1.0"/>
-    <limit lower="-${2*pi}" upper="${2*pi}" effort="0.0" velocity="0.0"/>
-</joint>
-<link name="l1">
-     <inertial>
-			<origin xyz="0.0 0.0 +0.25" rpy="0 0 0"/>
-			<mass value="1e+00"/>
-			<inertia
-            ixx="1.3778118e-01" ixy="5.1395441e-06" ixz="2.1163457e-04"
-            iyx="5.1395441e-06" iyy="1.3826689e-01" iyz="1.1751288e-02"
-            izx="2.1163457e-04" izy="1.1751288e-02" izz="3.5020186e-02"/>
-	</inertial>
-    <visual>
-        <geometry>
-            <cylinder radius="0.03" length="0.2"/>
-        </geometry>
-        <origin xyz="0.0 0.0 0.1" rpy="0.0 0.0 0.0"/>
-        <material name="silver"/>
-    </visual>
-    <!-- Add a sphere to create a curved joint -->
-    <visual>
-      <geometry>
-        <sphere radius="0.035"/>
-      </geometry>
-      <origin xyz="0.0 0.0 0.2" rpy="0.0 0.0 0.0"/>
-      <material name="gray"/>
-    </visual>
-</link>
-<!-- Dummy Joint -->
-<joint name="j_dummy_1_2" type="fixed">
-    <origin xyz="0.0 0.0 0.2" rpy="0.0 0.0 0.0"/>
+<?xml version="1.0" ?>
+<robot name="six-axis" xmlns:ros2_control="http://www.ros.org/wiki/ros2_control">
+    <material name="gray">
+        <color rgba="0.75 0.75 0.75 1.0"/>
+    </material>
+    <material name="silver">
+        <color rgba="0.9 0.9 0.98 1.0"/>
+    </material>
+    <!-- Base Link -->
+    <link name="base_link">
+        <!-- <visual>
+            <geometry>
+                <box size="0.40 0.40 0.12"/>
+            </geometry>
+            <origin xyz="0 0 0"/>
+            <material name="gray"/>
+        </visual>
+        <collision>
+            <geometry>
+                <box size="0.40 0.40 0.12"/>
+            </geometry>
+            <origin xyz="0 0 0"/>
+        </collision>
+        <inertial>
+            <origin xyz="0 0 0.06"/>
+            <mass value="20.0"/>
+            <inertia
+                ixx="0.25" ixy="0.0" ixz="0.0"
+                iyy="0.25" iyz="0.0"
+                izz="0.25"/>
+        </inertial> -->
+    </link>
+    <!-- j0 -->
+    <joint name="j0" type="fixed">
+        <origin rpy="0.0 0.0 0.0" xyz="0.0 0.0 0.0"/>
+        <parent link="base_link"/>
+        <child link="l0"/>
+        <axis xyz="0.0 0.0 0.0"/>
+        <limit effort="0.0" lower="0.0" upper="0.0" velocity="0.0"/>
+    </joint>
+    <link name="l0">
+        <inertial>
+            <origin xyz="0 0 0.025"/>
+            <mass value="12.0"/>
+            <inertia
+                ixx="0.004" ixy="0.0" ixz="0.0"
+                iyy="0.004" iyz="0.0"
+                izz="0.003"/>
+        </inertial>
+        <visual>
+            <geometry>
+                <cylinder length="0.05" radius="0.1"/>
+            </geometry>
+            <origin rpy="0.0 0.0 0.0" xyz="0.0 0.0 0.0"/>
+            <material name="silver"/>
+        </visual>
+        <collision>
+            <geometry>
+                <cylinder length="0.05" radius="0.1"/>
+            </geometry>
+            <origin rpy="0.0 0.0 0.0" xyz="0.0 0.0 0.0"/>
+        </collision>
+    </link>
+    <!-- j1 -->
+    <joint name="j1" type="revolute">
+        <origin rpy="0.0 0.0 0.0" xyz="0.0 0.0 0.0"/>
+        <parent link="l0"/>
+        <child link="l1"/>
+        <axis xyz="0.0 0.0 1.0"/>
+        <limit effort="20.0" lower="-6.283185307179586" upper="6.283185307179586" velocity="2.0"/>
+        <dynamics damping="0.2" friction="0.05"/>
+    </joint>
+    <link name="l1">
+        <inertial>
+        <origin xyz="0 0 0.1"/>
+        <mass value="2.5"/>
+        <inertia
+            ixx="0.010" ixy="0.0" ixz="0.0"
+            iyy="0.010" iyz="0.0"
+            izz="0.006"/>
+        </inertial>
+        <visual>
+            <geometry>
+                <cylinder length="0.2" radius="0.03"/>
+            </geometry>
+            <origin rpy="0.0 0.0 0.0" xyz="0.0 0.0 0.1"/>
+            <material name="silver"/>
+        </visual>
+        <visual>
+            <geometry>
+                <sphere radius="0.035"/>
+            </geometry>
+            <origin rpy="0.0 0.0 0.0" xyz="0.0 0.0 0.2"/>
+            <material name="gray"/>
+        </visual>
+        <collision>
+            <geometry>
+                <cylinder length="0.2" radius="0.03"/>
+            </geometry>
+            <origin rpy="0.0 0.0 0.0" xyz="0.0 0.0 0.1"/>
+        </collision>
+        <collision>
+            <geometry>
+                <sphere radius="0.035"/>
+            </geometry>
+            <origin rpy="0.0 0.0 0.0" xyz="0.0 0.0 0.2"/>
+        </collision>
+    </link>
+  <!-- Dummy l1 and l2 -->
+  <joint name="j_dummy_1_2" type="fixed">
+    <origin rpy="0.0 0.0 0.0" xyz="0.0 0.0 0.2"/>
     <parent link="l1"/>
     <child link="l2"/>
-</joint>
-<link name="l2">
-     <inertial>
-			<origin xyz="0.25 0.0 0.0" rpy="0 0 0"/>
-			<mass value="1e+00"/>
-			<inertia
-				ixx="3.0406895e-01" ixy="5.6383979e-04" ixz="4.4113010e-01"
-				iyx="5.6383979e-04" iyy="1.9934350e+00" iyz="1.2111129e-06"
-				izx="4.4113010e-01" izy="1.2111129e-06" izz="1.7471456e+00"/>
-	</inertial>
-    <visual>
-        <geometry>
-            <cylinder radius="0.03" length="0.25"/>
-        </geometry>
-        <origin xyz="0.125 0.0 0.0" rpy="0.0 ${pi/2} 0.0"/>
-        <material name="silver"/>
-    </visual>
-    <!-- Add a sphere to create a curved joint -->
-    <visual>
-      <geometry>
-        <sphere radius="0.035"/>
-      </geometry>
-      <origin xyz="0.25 0.0 0.0" rpy="0.0 0.0 0.0"/>
-      <material name="gray"/>
-    </visual>
-</link>
-<joint name="j2" type="revolute">
-    <origin xyz="0.25 0.0 0.0" rpy="0.0 ${pi/2} 0.0"/>
+  </joint>
+  <link name="l2">
+    <inertial>
+    <origin xyz="0.125 0 0"/>
+    <mass value="3.0"/>
+    <inertia
+        ixx="0.022" ixy="0.0" ixz="0.0"
+        iyy="0.030" iyz="0.0"
+        izz="0.015"/>
+    </inertial>
+    <visual>
+      <geometry>
+        <cylinder length="0.25" radius="0.03"/>
+      </geometry>
+      <origin rpy="0.0 1.5707963267948966 0.0" xyz="0.125 0.0 0.0"/>
+      <material name="silver"/>
+    </visual>
+    <visual>
+      <geometry>
+        <sphere radius="0.035"/>
+      </geometry>
+      <origin rpy="0.0 0.0 0.0" xyz="0.25 0.0 0.0"/>
+      <material name="gray"/>
+    </visual>
+    <collision>
+      <geometry>
+        <cylinder length="0.25" radius="0.03"/>
+      </geometry>
+      <origin rpy="0.0 1.5707963267948966 0.0" xyz="0.125 0.0 0.0"/>
+    </collision>
+    <collision>
+      <geometry>
+        <sphere radius="0.035"/>
+      </geometry>
+      <origin rpy="0.0 0.0 0.0" xyz="0.25 0.0 0.0"/>
+    </collision>
+  </link>
+  <!-- j2 -->
+  <joint name="j2" type="revolute">
+    <origin rpy="0.0 1.5707963267948966 0.0" xyz="0.25 0.0 0.0"/>
     <parent link="l2"/>
     <child link="l3"/>
     <axis xyz="0.0 0.0 1.0"/>
-    <limit lower="${-pi/2}" upper="${pi/2}" effort="0.0" velocity="0.0"/>
-</joint>
-<link name="l3">
-     <inertial>
-			<origin xyz="-0.15 0.0 0.0" rpy="0 0 0"/>
-			<mass value="3e+00"/>
-			<inertia
-				ixx="3.1982320e-02" ixy="-1.5528529e-05" ixz="-4.8994800e-05"
-				iyx="-1.5528529e-05" iyy="2.8261283e-02" iyz="7.1406845e-03"
-				izx="-4.8994800e-05" izy="7.1406845e-03" izz="8.8063347e-03"/>
-	</inertial>
-    <visual>
-        <geometry>
-            <cylinder radius="0.03" length="0.3"/>
-        </geometry>
-        <origin xyz="-0.15 0.0 0.0 " rpy="0.0  ${pi/2} 0.0"/>
-        <material name="silver"/>
-    </visual>
-    <!-- Add a sphere to create a curved joint -->
-    <visual>
-      <geometry>
-        <sphere radius="0.035"/>
-      </geometry>
-      <origin xyz="0.0 0.0 0.0" rpy="0.0 0.0 0.0"/>
-      <material name="gray"/>
-    </visual>
-</link>
-<joint name="j3" type="revolute">
-    <origin xyz="-0.30 0.0 0.0" rpy="0.0 0.0 0.0"/>
+    <limit effort="20.0" lower="-1.5707963267948966" upper="1.5707963267948966" velocity="2.0"/>
+    <dynamics damping="0.2" friction="0.05"/>
+  </joint>
+  <link name="l3">
+    <inertial>
+    <origin xyz="-0.15 0 0"/>
+    <mass value="2.5"/>
+    <inertia
+        ixx="0.015" ixy="0.0" ixz="0.0"
+        iyy="0.020" iyz="0.0"
+        izz="0.010"/>
+    </inertial>
+    <visual>
+      <geometry>
+        <cylinder length="0.3" radius="0.03"/>
+      </geometry>
+      <origin rpy="0.0 1.5707963267948966 0.0" xyz="-0.15 0.0 0.0"/>
+      <material name="silver"/>
+    </visual>
+    <visual>
+      <geometry>
+        <sphere radius="0.035"/>
+      </geometry>
+      <origin rpy="0.0 0.0 0.0" xyz="0.0 0.0 0.0"/>
+      <material name="gray"/>
+    </visual>
+    <collision>
+      <geometry>
+        <cylinder length="0.3" radius="0.03"/>
+      </geometry>
+      <origin rpy="0.0 1.5707963267948966 0.0" xyz="-0.15 0.0 0.0"/>
+    </collision>
+    <collision>
+      <geometry>
+        <sphere radius="0.035"/>
+      </geometry>
+      <origin rpy="0.0 0.0 0.0" xyz="0.0 0.0 0.0"/>
+    </collision>
+  </link>
+  <!-- j3 -->
+  <joint name="j3" type="revolute">
+    <origin rpy="0.0 0.0 0.0" xyz="-0.30 0.0 0.0"/>
     <parent link="l3"/>
     <child link="l4"/>
     <axis xyz="0.0 0.0 1.0"/>
-    <limit lower="${-pi/2}" upper="${pi/2}" effort="0.0" velocity="0.0"/>
-</joint>
-<link name="l4">
-     <inertial>
-			<origin xyz="0.0 0.0 -0.12" rpy="0 0 0"/>
-			<mass value="1e+00"/>
-			<inertia
-				ixx="3.0406895e-01" ixy="5.6383979e-04" ixz="4.4113010e-01"
-				iyx="5.6383979e-04" iyy="1.9934350e+00" iyz="1.2111129e-06"
-				izx="4.4113010e-01" izy="1.2111129e-06" izz="1.7471456e+00"/>
-	</inertial>
-    <visual>
-        <geometry>
-            <cylinder radius="0.03" length="0.24"/>
-        </geometry>
-        <origin xyz="0.0 0.0 -0.12" rpy="0.0 0.0 0.0"/>
-        <material name="silver"/>
-    </visual>
-    <!-- Add a sphere to create a curved joint -->
-    <visual>
-      <geometry>
-        <sphere radius="0.035"/>
-      </geometry>
-      <origin xyz="0.0 0.0 0.0" rpy="0.0 0.0 0.0"/>
-      <material name="gray"/>
-    </visual>
-</link>
-<!-- Dummy Joint -->
-<joint name="j_dummy" type="fixed">
-    <origin xyz="0.0 0.0 -0.24" rpy="0.0 0.0 0.0"/>
+    <limit effort="20.0" lower="-1.5707963267948966" upper="1.5707963267948966" velocity="2.0"/>
+    <dynamics damping="0.2" friction="0.05"/>
+  </joint>
+  <link name="l4">
+    <inertial>
+    <origin xyz="0 0 -0.12"/>
+    <mass value="1.2"/>
+    <inertia
+        ixx="0.004" ixy="0.0" ixz="0.0"
+        iyy="0.006" iyz="0.0"
+        izz="0.003"/>
+    </inertial>
+    <visual>
+      <geometry>
+        <cylinder length="0.24" radius="0.03"/>
+      </geometry>
+      <origin rpy="0.0 0.0 0.0" xyz="0.0 0.0 -0.12"/>
+      <material name="silver"/>
+    </visual>
+    <visual>
+      <geometry>
+        <sphere radius="0.035"/>
+      </geometry>
+      <origin rpy="0.0 0.0 0.0" xyz="0.0 0.0 0.0"/>
+      <material name="gray"/>
+    </visual>
+    <collision>
+      <geometry>
+        <cylinder length="0.24" radius="0.03"/>
+      </geometry>
+      <origin rpy="0.0 0.0 0.0" xyz="0.0 0.0 -0.12"/>
+    </collision>
+    <collision>
+      <geometry>
+        <sphere radius="0.035"/>
+      </geometry>
+      <origin rpy="0.0 0.0 0.0" xyz="0.0 0.0 0.0"/>
+    </collision>
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
Commit message: Everything works in RViz

File: arm_ws/src/arm_description/urdf/arm.urdf.xacro (robot description, xacro)
@@ -4,4 +4,16 @@
   xmlns:xacro="http://www.ros.org/wiki/xacro"
   xmlns:ros2_control="http://www.ros.org/wiki/ros2_control">
+  <xacro:macro name="simple_transmission" params="joint">
+    <transmission name="${joint}_trans">
+      <type>transmission_interface/SimpleTransmission</type>
+      <joint name="${joint}">
+        <hardwareInterface>hardware_interface/PositionJointInterface</hardwareInterface>
+      </joint>
+      <actuator name="${joint}_motor">
+        <hardwareInterface>hardware_interface/PositionJointInterface</hardwareInterface>
+        <mechanicalReduction>1</mechanicalReduction>
+      </actuator>
+    </transmission>
+  </xacro:macro>
     <material name="gray">
         <color rgba="0.75 0.75 0.75 1.0"/>
@@ -522,3 +534,12 @@
   </joint>
   <xacro:include filename="six-axis.ros2_control.xacro" />
+  <xacro:include filename="$(find arm_gazebo)/urdf/gazebo_plugins.xacro"/>
+  <xacro:add_gazebo_plugins/>
+  <xacro:simple_transmission joint="j1"/>
+  <xacro:simple_transmission joint="j2"/>
+  <xacro:simple_transmission joint="j3"/>
+  <xacro:simple_transmission joint="j4"/>
+  <xacro:simple_transmission joint="j5"/>
+  <xacro:simple_transmission joint="j6"/>
+  <xacro:simple_transmission joint="gripper_right_finger_joint"/>
 </robot>

File: arm_ws/src/arm_description/urdf/six-axis.ros2_control.xacro (robot description, xacro)
@@ -3,7 +3,32 @@
         <ros2_control name="six_axis_arm" type="system">
             <hardware>
-                <!-- By default, set up controllers for simulation. This won't work on real hardware -->
-                <plugin>mock_components/GenericSystem</plugin>
+              <plugin>gz_ros2_control/GazeboSimSystem</plugin>
             </hardware>
+              <!--
+                  MODIFY NOTE (Gazebo Integration):
+                    FROM:
+                      <plugin>mock_components/GenericSystem</plugin>
+                    TO:
+                      <plugin>gz_ros2_control/GazeboSimSystem</plugin>
+                    WHY:
+                     - mock_components/GenericSystem is a FAKE hardware interface.
+                     - It only works for RViz and MoveIt visualization (no physics).
+                     - Gazebo requires a REAL simulation hardware interface to:
+                       • expose joint state interfaces
+                       • expose command interfaces
+                       • connect controllers to physics
+                     - gz_ros2_control/GazeboSimSystem is the official hardware plugin
+                       that bridges:
+                         ros2_control  ↔  Gazebo Sim (gz)
+                    WITHOUT THIS CHANGE:
+                     - Controllers load but cannot activate
+                     - Errors like:
+                       "No state interfaces found"
+                       "command interface j1/position is not available"
+                    WITH THIS CHANGE:
+                     - Gazebo publishes joint states
+                     - Controllers activate successfully
+                     - Arm moves physically in Gazebo
+                                                     -->
             <joint name="j1">
                 <command_interface name="position"/>

File: arm_ws/src/arm_gazebo/urdf/gazebo_plugins.xacro (robot description, xacro)
@@ -1,15 +1,12 @@
 <?xml version="1.0"?>
-<xacro:macro name="add_gazebo_plugins" params=""
-    xmlns:xacro="http://www.ros.org/wiki/xacro">
-  <gazebo>
-    <plugin
-      filename="libgz_ros2_control-system.so"
-      name="gz_ros2_control::GazeboSystem">
-      <parameters>
-        <ros2_control_config>
-          $(find arm_bringup)/config/ros2_controllers.yaml
-        </ros2_control_config>
-      </parameters>
-    </plugin>
-  </gazebo>
-</xacro:macro>
+<robot xmlns:xacro="http://www.ros.org/wiki/xacro">
+  <xacro:macro name="add_gazebo_plugins">
+    <gazebo>
+      <plugin
+        filename="libgz_ros2_control-system.so"
+        name="gz_ros2_control::GazeboSimROS2ControlPlugin">
+        <parameters>$(find arm_bringup)/config/ros2_controllers.yaml</parameters>
+      </plugin>
+    </gazebo>
+  </xacro:macro>
+</robot>

Commit message: its now started to work

File: arm_ws/src/arm_description/urdf/arm.urdf.xacro (robot description, xacro)
@@ -57,5 +57,5 @@
         <inertial>
             <origin xyz="0 0 0.025"/>
-            <mass value="12.0"/>
+            <mass value="100.0"/>
             <inertia
                 ixx="0.004" ixy="0.0" ixz="0.0"

Commit message: Moveit2 mostly done

File: arm_ws/src/arm_description/urdf/arm.urdf.xacro (robot description, xacro)
@@ -89,5 +89,5 @@
         <inertial>
         <origin xyz="0 0 0.1"/>
-        <mass value="2.5"/>
+        <mass value="3"/>
         <inertia
             ixx="0.010" ixy="0.0" ixz="0.0"
@@ -131,5 +131,5 @@
     <inertial>
     <origin xyz="0.125 0 0"/>
-    <mass value="3.0"/>
+    <mass value="2.5"/>
     <inertia
         ixx="0.022" ixy="0.0" ixz="0.0"
@@ -170,11 +170,11 @@
     <child link="l3"/>
     <axis xyz="0.0 0.0 1.0"/>
-    <limit effort="20.0" lower="-1.5707963267948966" upper="1.5707963267948966" velocity="2.0"/>
-    <dynamics damping="0.2" friction="0.05"/>
+    <limit effort="30.0" lower="-1.5707963267948966" upper="1.5707963267948966" velocity="2.0"/>
+    <dynamics damping="0.2" friction="0.08"/>
   </joint>
   <link name="l3">
     <inertial>
     <origin xyz="-0.15 0 0"/>
-    <mass value="2.5"/>
+    <mass value="2.2"/>
     <inertia
         ixx="0.015" ixy="0.0" ixz="0.0"

Commit message: Just Before MTC

File: arm_ws/src/arm_description/urdf/arm.urdf.xacro (robot description, xacro)
@@ -529,7 +529,7 @@
   <link name="tool0"/>
   <joint name="g_base_to_tool0" type="fixed">
-    <origin xyz="0 0 0.15" rpy="0 0 0"/>
-    <parent link="g_base"/>
-    <child link="tool0"/>
+      <origin xyz="0 0 0.03" rpy="0 0 0"/>
+      <parent link="g_base"/>
+      <child link="tool0"/>
   </joint>
   <xacro:include filename="six-axis.ros2_control.xacro" />

Commit message: Task3: Effort-based gripper working with stable grasp

File: arm_ws/src/arm_description/urdf/arm.urdf.xacro (robot description, xacro)
@@ -16,4 +16,16 @@
     </transmission>
   </xacro:macro>
+  <xacro:macro name="effort_transmission" params="joint">
+  <transmission name="${joint}_effort_trans">
+    <type>transmission_interface/SimpleTransmission</type>
+    <joint name="${joint}">
+      <hardwareInterface>hardware_interface/EffortJointInterface</hardwareInterface>
+    </joint>
+    <actuator name="${joint}_motor">
+      <hardwareInterface>hardware_interface/EffortJointInterface</hardwareInterface>
+      <mechanicalReduction>1</mechanicalReduction>
+    </actuator>
+  </transmission>
+</xacro:macro>
     <material name="gray">
         <color rgba="0.75 0.75 0.75 1.0"/>
@@ -529,5 +541,5 @@
   <link name="tool0"/>
   <joint name="g_base_to_tool0" type="fixed">
-      <origin xyz="0 0 0.03" rpy="0 0 0"/>
+      <origin xyz="0 0 0.13" rpy="0 0 0"/>
       <parent link="g_base"/>
       <child link="tool0"/>
@@ -542,4 +554,17 @@
   <xacro:simple_transmission joint="j5"/>
   <xacro:simple_transmission joint="j6"/>
-  <xacro:simple_transmission joint="gripper_right_finger_joint"/>
+  <!-- <xacro:simple_transmission joint="gripper_right_finger_joint"/> -->
+  <xacro:effort_transmission joint="gripper_right_finger_joint"/>
+  <gazebo reference="gripper_left_finger">
+    <mu1>2.0</mu1>
+    <mu2>2.0</mu2>
+    <kp>100000</kp>
+    <kd>10</kd>
+  </gazebo>
+  <gazebo reference="gripper_right_finger">
+    <mu1>2.0</mu1>
+    <mu2>2.0</mu2>
+    <kp>100000</kp>
+    <kd>10</kd>
+  </gazebo>
 </robot>

File: arm_ws/src/arm_description/urdf/six-axis.ros2_control.xacro (robot description, xacro)
@@ -74,9 +74,8 @@
             </joint>
             <joint name="gripper_right_finger_joint">
-                <command_interface name="position"/>
-                <state_interface name="position">
-                  <param name="initial_value">0.0</param>
-                </state_interface>
-                <state_interface name="velocity"/>
+              <command_interface name="effort"/>
+              <state_interface name="position"/>
+              <state_interface name="velocity"/>
+              <state_interface name="effort"/>
             </joint>
         </ros2_control>

Commit message: 2025 comes to an end

File: arm_ws/src/arm_description/urdf/arm.urdf.xacro (robot description, xacro)
@@ -445,5 +445,5 @@
   <!-- Connect wrist to gripper base -->
   <joint name="le_1_to_g_base" type="fixed">
-    <origin rpy="0 0 0" xyz="0 0 0.1"/>
+    <origin xyz="0 0 0.10"/>
     <parent link="le_1"/>
     <child link="g_base"/>
@@ -541,7 +541,7 @@
   <link name="tool0"/>
   <joint name="g_base_to_tool0" type="fixed">
-      <origin xyz="0 0 0.13" rpy="0 0 0"/>
-      <parent link="g_base"/>
-      <child link="tool0"/>
+    <origin xyz="0 0 0.03" rpy="3.14159 0 0"/>
+    <parent link="g_base"/>
+    <child link="tool0"/>
   </joint>
   <xacro:include filename="six-axis.ros2_control.xacro" />
